Commit message: Major updates to hardware interface and URDF configuration
- Updated hardware interface (hpp/cpp) for improved motor control
- Refined URDF and ros2_control configuration
- Updated controller parameters for better performance
- Updated LiDAR and navigation configurations

File: ros2_ws/src/dummybot_bringup/description/urdf/dummybot.ros2_control.xacro (robot description, xacro)
@@ -1,22 +1,41 @@
 <?xml version="1.0"?>
 <robot xmlns:xacro="http://www.ros.org/wiki/xacro">
-  <xacro:macro name="dummybot_ros2_control" params="
-    name
-    serial_port
-    serial_baud
-    wheel_radius
-    wheel_separation
-    ticks_per_revolution">
+  <xacro:macro name="dummybot_ros2_control" params="name prefix
+                                                     serial_port
+                                                     serial_baud
+                                                     wheel_radius
+                                                     wheel_separation
+                                                     ticks_per_revolution
+                                                     pid_kp
+                                                     pid_kd
+                                                     pid_ki
+                                                     pid_ko
+                                                     calibration_fl
+                                                     calibration_fr
+                                                     calibration_rl
+                                                     calibration_rr">
     <ros2_control name="${name}" type="system">
       <hardware>
         <plugin>dummybot_hardware/DummyBotHardwareInterface</plugin>
+        <!-- Serial Communication Parameters -->
         <param name="serial_port">${serial_port}</param>
         <param name="serial_baud">${serial_baud}</param>
+        <!-- Robot Physical Parameters -->
         <param name="wheel_radius">${wheel_radius}</param>
         <param name="wheel_separation">${wheel_separation}</param>
         <param name="ticks_per_revolution">${ticks_per_revolution}</param>
+        <!-- PID Controller Parameters (INT, ordine: kp kd ki ko) -->
+        <param name="pid_kp">${pid_kp}</param>
+        <param name="pid_kd">${pid_kd}</param>
+        <param name="pid_ki">${pid_ki}</param>
+        <param name="pid_ko">${pid_ko}</param>
+        <!-- Calibration Factors (FLOAT) -->
+        <param name="calibration_fl">${calibration_fl}</param>
+        <param name="calibration_fr">${calibration_fr}</param>
+        <param name="calibration_rl">${calibration_rl}</param>
+        <param name="calibration_rr">${calibration_rr}</param>
       </hardware>
-      <!-- Front Left Wheel -->
-      <joint name="front_left_wheel_joint">
+      <!-- Front Left Wheel Joint -->
+      <joint name="${prefix}front_left_wheel_joint">
         <command_interface name="velocity">
           <param name="min">-10</param>
@@ -26,6 +45,6 @@
         <state_interface name="velocity"/>
       </joint>
-      <!-- Front Right Wheel -->
-      <joint name="front_right_wheel_joint">
+      <!-- Front Right Wheel Joint -->
+      <joint name="${prefix}front_right_wheel_joint">
         <command_interface name="velocity">
           <param name="min">-10</param>
@@ -35,6 +54,6 @@
         <state_interface name="velocity"/>
       </joint>
-      <!-- Rear Left Wheel -->
-      <joint name="rear_left_wheel_joint">
+      <!-- Rear Left Wheel Joint -->
+      <joint name="${prefix}rear_left_wheel_joint">
         <command_interface name="velocity">
           <param name="min">-10</param>
@@ -44,6 +63,6 @@
         <state_interface name="velocity"/>
       </joint>
-      <!-- Rear Right Wheel -->
-      <joint name="rear_right_wheel_joint">
+      <!-- Rear Right Wheel Joint -->
+      <joint name="${prefix}rear_right_wheel_joint">
         <command_interface name="velocity">
           <param name="min">-10</param>

File: ros2_ws/src/dummybot_bringup/description/urdf/dummybot.urdf.xacro (robot description, xacro)
@@ -49,7 +49,17 @@
   <xacro:property name="lidar_z_offset" value="0.1775"/>   <!-- 17.75cm deasupra base_chassis -->
   <!-- ESP32 Hardware Interface -->
-  <xacro:property name="serial_port" value="/dev/ttyESP32"/>
+  <xacro:property name="serial_port" value="/dev/ttyUSB0"/>
   <xacro:property name="serial_baud" value="115200"/>
   <xacro:property name="ticks_per_revolution" value="1245"/>
+  <!-- PID Controller Parameters (INT pentru ESP32, ordine: kp kd ki ko) -->
+  <xacro:property name="pid_kp" value="300"/>
+  <xacro:property name="pid_kd" value="70"/>
+  <xacro:property name="pid_ki" value="0"/>
+  <xacro:property name="pid_ko" value="14"/>
+  <!-- Calibration Factors (FLOAT) -->
+  <xacro:property name="calibration_fl" value="0.875"/>
+  <xacro:property name="calibration_fr" value="1.065"/>
+  <xacro:property name="calibration_rl" value="1.025"/>
+  <xacro:property name="calibration_rr" value="1.025"/>
   <!-- Materials -->
   <material name="black">
@@ -209,8 +219,17 @@
   <xacro:dummybot_ros2_control
     name="DummyBotSystem"
+    prefix=""
     serial_port="${serial_port}"
     serial_baud="${serial_baud}"
     wheel_radius="${wheel_radius}"
     wheel_separation="${track_width}"
-    ticks_per_revolution="${ticks_per_revolution}"/>
+    ticks_per_revolution="${ticks_per_revolution}"
+    pid_kp="${pid_kp}"
+    pid_kd="${pid_kd}"
+    pid_ki="${pid_ki}"
+    pid_ko="${pid_ko}"
+    calibration_fl="${calibration_fl}"
+    calibration_fr="${calibration_fr}"
+    calibration_rl="${calibration_rl}"
+    calibration_rr="${calibration_rr}"/>
 </robot>
