Commit message: feat: Integrate LD06 LiDAR with permanent USB mapping
- Add ldlidar_stl_ros2 driver as submodule (official LD06 driver)
- Configure udev rules for persistent /dev/ttyESP32 and /dev/ttyLIDAR
- Update dummybot.launch.py to include LiDAR
- Fix serial port configuration in URDF (use symlinks)
- Remove verbose motor logging from hardware interface
- Update .gitignore for build artifacts

Hardware:
- ESP32 on /dev/ttyESP32 (USB port usb2/2-1)
- LD06 LiDAR on /dev/ttyLIDAR (USB port usb4/4-2)

LiDAR publishes on /scan at 10 Hz
System fully operational for SLAM and autonomous navigation

File: ros2_ws/src/dummybot_bringup/description/urdf/dummybot.urdf.xacro (robot description, xacro)
@@ -14,5 +14,5 @@
   <xacro:property name="base_height" value="0.15"/>
   <!-- Serial configuration -->
-  <xacro:property name="serial_port" value="/dev/ttyUSB0"/>
+  <xacro:property name="serial_port" value="/dev/ttyESP32"/>
   <xacro:property name="serial_baud" value="115200"/>
   <xacro:property name="ticks_per_revolution" value="1760"/>

Commit message: feat: Add SLAM Toolbox integration with auto-activation
- Configure SLAM Toolbox for LD06 LiDAR mapping
- Add slam.launch.py with automatic lifecycle activation
- Configure mapper parameters (5cm resolution, loop closing)
- Fix base_frame from base_footprint to base_link
- Add map saving functionality
- Tested and functional on Raspberry Pi 5

File: ros2_ws/src/dummybot_bringup/description/urdf/dummybot.urdf.xacro (robot description, xacro)
@@ -6,5 +6,5 @@
   <xacro:property name="use_mock_hardware" value="false"/>
   <!-- Robot dimensions (from ESP32 config.h) -->
-  <xacro:property name="wheel_radius" value="0.0325"/>        <!-- 65mm / 2 -->
+  <xacro:property name="wheel_radius" value="0.0345"/>        <!-- 69mm / 2 -->
   <xacro:property name="wheel_width" value="0.026"/>          <!-- 26mm width -->
   <xacro:property name="wheel_separation" value="0.3863"/>    <!-- Lx: 386.3mm -->

Commit message: Add autonomous navigation v1.2 with URDF fixes and navigation stack
Major changes:
- Fixed URDF robot orientation and coordinate system
- Corrected wheel joint rotation (rpy='0 pi/2 0', axis='0 0 1')
- Updated LiDAR positioning (centered laterally, on chassis top)
- Fixed diff_drive_controller stamped velocity configuration
- Updated wheel_separation and chassis dimensions
- Integrated SLAM Toolbox with proper remappings
- Updated Nav2 parameters for navigation stack
- Added LD19 LiDAR configuration and launch files
- Added camera and sensors launch files
- Added backup configurations (_v0 files)
- Added amr2ax_nav2 package with maps and waypoint navigation

File: ros2_ws/src/dummybot_bringup/description/urdf/dummybot.urdf.xacro (robot description, xacro)
@@ -5,21 +5,51 @@
   <!-- Properties -->
   <xacro:property name="use_mock_hardware" value="false"/>
-  <!-- Robot dimensions - După rotație 90°: X=lateral, Y=față-spate -->
-  <xacro:property name="wheel_radius" value="0.0345"/>
-  <xacro:property name="wheel_width" value="0.028"/>
-  <xacro:property name="wheelbase" value="0.374"/>            <!-- Track width (lateral X) -->
-  <xacro:property name="wheel_separation" value="0.390"/>     <!-- Wheelbase (longitudinal Y) -->
-  <xacro:property name="base_length" value="0.36"/>           <!-- X (scurt, lateral) -->
-  <xacro:property name="base_width" value="0.46"/>            <!-- Y (lung, față-spate) -->
-  <xacro:property name="base_height" value="0.14"/>
-  <xacro:property name="ground_clearance" value="0.0345"/>
-  <xacro:property name="wheel_z_offset" value="-0.02"/>
-  <!-- Poziții roți pe Y (față-spate) -->
-  <xacro:property name="front_wheel_y_offset" value="0.175"/>
-  <xacro:property name="rear_wheel_y_offset" value="-0.215"/>
-  <!-- Serial configuration -->
+  <!-- ============================================ -->
+  <!-- DIMENSIUNI FIZICE REALE - SISTEM ROS STANDARD -->
+  <!-- X = înainte (FAȚĂ) = 36cm (ce tu numești "lățime") -->
+  <!-- Y = lateral (STÂNGA-DREAPTA) = 46.5cm (ce tu numești "lungime") -->
+  <!-- Z = sus (vertical) -->
+  <!-- ============================================ -->
+  <!-- Roți -->
+  <xacro:property name="wheel_radius" value="0.0345"/>     <!-- 69mm diametru / 2 -->
+  <xacro:property name="wheel_width" value="0.028"/>       <!-- 28mm grosime -->
+  <!-- Distanțe între roți -->
+  <xacro:property name="wheelbase" value="0.400"/>         <!-- FR-FL distanță FAȚĂ-SPATE (37.4cm) -->
+  <xacro:property name="track_width" value="0.390"/>       <!-- FR-RR distanță LATERALĂ (39cm) -->
+  <!-- Chassis -->
+  <xacro:property name="chassis_length" value="0.470"/>    <!-- 36cm pe X (față-spate, "lățimea" ta) -->
+  <xacro:property name="chassis_width" value="0.365"/>     <!-- 46.5cm pe Y (lateral, "lungimea" ta) -->
+  <xacro:property name="chassis_height" value="0.150"/>    <!-- 16cm înălțime (Z) -->
+  <xacro:property name="ground_clearance" value="0.060"/>  <!-- 5cm de la sol la baza chassis -->
+  <!-- Poziționare roți față de chassis -->
+  <!-- FR/FL la 5cm de față → +36/2 - 5 = +13cm = +0.13m -->
+  <!-- RR/RL la 3cm de spate → -36/2 + 3 = -15cm = -0.15m -->
+  <!-- Verificare: 13cm + 15cm = 28cm (ar trebui ~37.4cm pentru wheelbase) -->
+  <!-- Corectie: 5cm față, 32.4cm spate? Sau 18.7cm față, 18.7cm spate? -->
+  <!-- Să recalculăm cu wheelbase = 37.4cm: -->
+  <!-- Centru roți față: +37.4/2 = +18.7cm -->
+  <!-- Centru roți spate: -37.4/2 = -18.7cm -->
+  <xacro:property name="front_wheel_x" value="0.195"/>     <!-- +18.7cm -->
+  <xacro:property name="rear_wheel_x" value="-0.195"/>     <!-- -18.7cm -->
+  <xacro:property name="left_wheel_y" value="-0.200"/>     <!-- +18.7cm -->
+  <xacro:property name="right_wheel_y" value="0.200"/>     <!-- -18.7cm -->
+  <!-- Offset vertical roți: centru la 5.8cm de sol, minus ground_clearance de 5cm -->
+  <xacro:property name="wheel_z_offset" value="0.008"/>    <!-- 5.8cm - 5cm = 0.8cm -->
+  <xacro:property name="lidar_len" value="0.037" />
+  <xacro:property name="lidar_radius" value="0.018" />
+  <xacro:property name="lidar_mass" value="0.015" />
+  <!-- LiDAR poziționare -->
+  <!-- "12cm de la fața carcasei până la început LiDAR" -->
+  <!-- Dacă fața chassis e la +18cm, iar LiDAR începe la +12cm de la față... -->
+  <!-- Stai, trebuie clarificat: 12cm de la MARGINEA chassis sau de la CENTRU? -->
+  <!-- Presupun: 12cm de la MARGINEA din față (la +18cm) -->
+  <!-- Deci început LiDAR = +18cm - 12cm = +6cm de la centru -->
+  <!-- Centru LiDAR = +6cm + 1.9cm (jumătate) = +7.9cm = 0.079m -->
+  <xacro:property name="lidar_x_offset" value="0.079"/>    <!-- 7.9cm înainte de centru -->
+  <xacro:property name="lidar_z_offset" value="0.1775"/>   <!-- 17.75cm deasupra base_chassis -->
+  <!-- ESP32 Hardware Interface -->
   <xacro:property name="serial_port" value="/dev/ttyESP32"/>
   <xacro:property name="serial_baud" value="115200"/>
-  <xacro:property name="ticks_per_revolution" value="1760"/>
+  <xacro:property name="ticks_per_revolution" value="1245"/>
   <!-- Materials -->
   <material name="black">
@@ -32,29 +62,32 @@
     <color rgba="0.8 0.0 0.0 1.0"/>
   </material>
-  <!-- Base Footprint -->
-  <link name="base_footprint"/>
-  <joint name="base_footprint_joint" type="fixed">
-    <parent link="base_footprint"/>
-    <child link="base_link"/>
-    <!-- MODIFICAT: Rotație 90° pe Z + ridicare deasupra solului -->
-    <origin xyz="0 0 ${ground_clearance}" rpy="0 0 ${-pi/2}"/>
+  <!-- ============================================ -->
+  <!-- BASE LINK (ROOT FRAME) -->
+  <!-- ============================================ -->
+  <link name="base_link"/>
+  <joint name="base_link_chassis_joint" type="fixed">
+    <parent link="base_link"/>
+    <child link="base_chassis"/>
+    <origin xyz="0 0 ${ground_clearance + chassis_height/2}" rpy="0 0 0"/>
   </joint>
-  <!-- Base Link -->
-  <link name="base_link">
+  <!-- ============================================ -->
+  <!-- BASE CHASSIS -->
+  <!-- ============================================ -->
+  <link name="base_chassis">
     <visual>
-      <origin xyz="0 0 ${base_height/2}" rpy="0 0 0"/>
-      <geometry>
-        <box size="${base_length} ${base_width} ${base_height}"/>
+      <origin xyz="0 0 0" rpy="0 0 0"/>
+      <geometry>
+        <box size="${chassis_length} ${chassis_width} ${chassis_height}"/>
       </geometry>
       <material name="dark_grey"/>
     </visual>
     <collision>
-      <origin xyz="0 0 ${base_height/2}" rpy="0 0 0"/>
-      <geometry>
-        <box size="${base_length} ${base_width} ${base_height}"/>
+      <origin xyz="0 0 0" rpy="0 0 0"/>
+      <geometry>
+        <box size="${chassis_length} ${chassis_width} ${chassis_height}"/>
       </geometry>
     </collision>
     <inertial>
-      <origin xyz="0 0 ${base_height/2}" rpy="0 0 0"/>
+      <origin xyz="0 0 0" rpy="0 0 0"/>
       <mass value="5.0"/>
       <inertia ixx="0.0833" ixy="0.0" ixz="0.0"
@@ -63,9 +96,12 @@
     </inertial>
   </link>
-  <!-- Wheel Macro -->
+  <!-- ============================================ -->
+  <!-- WHEEL MACRO -->
+  <!-- ============================================ -->
   <xacro:macro name="wheel" params="prefix x y">
     <link name="${prefix}_wheel_link">
       <visual>
-        <origin xyz="0 0 0" rpy="0 ${pi/2} 0"/>
+        <!-- FĂRĂ rotație aici -->
+        <origin xyz="0 0 0" rpy="${pi/2} 0 0"/>
         <geometry>
           <cylinder radius="${wheel_radius}" length="${wheel_width}"/>
@@ -74,5 +110,6 @@
       </visual>
       <collision>
-        <origin xyz="0 0 0" rpy="0 ${pi/2} 0"/>
+        <!-- FĂRĂ rotație aici -->
+        <origin xyz="0 0 0" rpy="${pi/2} 0 0"/>
         <geometry>
           <cylinder radius="${wheel_radius}" length="${wheel_width}"/>
@@ -80,9 +117,9 @@
       </collision>
       <inertial>
-        <origin xyz="0 0 0" rpy="0 0 0"/>
+        <origin xyz="0 0 0" rpy="${pi/2} 0 0"/>
         <mass value="0.5"/>
         <inertia ixx="0.0001" ixy="0.0" ixz="0.0"
-                 iyy="0.0001" iyz="0.0"
-                 izz="0.0001"/>
+                iyy="0.0001" iyz="0.0"
+                izz="0.0001"/>
       </inertial>
     </link>
@@ -90,43 +127,84 @@
       <parent link="base_link"/>
       <child link="${prefix}_wheel_link"/>
-      <origin xyz="${x} ${y} ${wheel_z_offset}" rpy="0 0 0"/>
-      <!-- MODIFICAT: Axa X pentru roți pe lateral -->
-      <axis xyz="1 0 0"/>
+      <!-- ROTAȚIE AICI în joint origin -->
+      <origin xyz="${x} ${y} ${wheel_radius}" rpy="0 0 0"/>
+      <!-- Axa Y = roata se rotește în jurul axei laterale -->
+      <axis xyz="0 1 0"/>
     </joint>
   </xacro:macro>
-  <!-- Instantiate 4 wheels - X=lateral, Y=față-spate -->
-  <xacro:wheel prefix="front_left"  x="${wheelbase/2}"   y="${front_wheel_y_offset}"/>
-  <xacro:wheel prefix="front_right" x="${-wheelbase/2}"  y="${front_wheel_y_offset}"/>
-  <xacro:wheel prefix="rear_left"   x="${wheelbase/2}"   y="${rear_wheel_y_offset}"/>
-  <xacro:wheel prefix="rear_right"  x="${-wheelbase/2}"  y="${rear_wheel_y_offset}"/>
-  <!-- LiDAR -->
-  <link name="laser_frame">
+  <!-- ============================================ -->
+  <!-- INSTANTIATE 4 WHEELS -->
+  <!-- FR = Front Right (față + dreapta, Y negativ) -->
+  <!-- FL = Front Left (față + stânga, Y pozitiv) -->
+  <!-- RR = Rear Right (spate + dreapta, Y negativ) -->
+  <!-- RL = Rear Left (spate + stânga, Y pozitiv) -->
+  <!-- ============================================ -->
+  <!-- CORECT: Swap X cu Y -->
+  <!-- Front Left (față + stânga) -->
+  <xacro:wheel prefix="front_left"  x="${front_wheel_x}"  y="${left_wheel_y}"/>
+  <!-- Front Right (față + dreapta) -->
+  <xacro:wheel prefix="front_right" x="${front_wheel_x}"  y="${right_wheel_y}"/>
+  <!-- Rear Left (spate + stânga) -->
+  <xacro:wheel prefix="rear_left"   x="${rear_wheel_x}"  y="${left_wheel_y}"/>
+  <!-- Rear Right (spate + dreapta) -->
+  <xacro:wheel prefix="rear_right"  x="${rear_wheel_x}"  y="${right_wheel_y}"/>
+  <!-- LIDAR LD19 Link -->
+  <link name="base_laser">
+    <collision>
+      <origin xyz="0 0 ${lidar_len/2}" rpy="0 0 0"/>
+      <geometry>
+        <cylinder length="${lidar_len}" radius="${lidar_radius}"/>
+      </geometry>
+    </collision>
     <visual>
-      <origin xyz="0 0 0" rpy="0 0 0"/>
-      <geometry>
-        <box size="0.035 0.035 0.035"/>
-      </geometry>
-      <material name="red"/>
+      <origin xyz="0 0 ${lidar_len/2}" rpy="0 0 0"/>
+      <geometry>
+        <cylinder length="${lidar_len}" radius="${lidar_radius}"/>
+      </geometry>
+      <material name="white"/>
     </visual>
-    <collision>
-      <origin xyz="0 0 0" rpy="0 0 0"/>
-      <geometry>
-        <box size="0.035 0.035 0.035"/>
-      </geometry>
-    </collision>
     <inertial>
-      <mass value="0.15"/>
-      <inertia ixx="0.0001" ixy="0.0" ixz="0.0"
-               iyy="0.0001" iyz="0.0"
-               izz="0.0001"/>
-    </inertial>
+      <origin xyz="0 0 ${lidar_len/2}  " rpy="0 0 0"/>
+      <mass value="${lidar_mass}"/>
+      <inertia
+        ixx="${lidar_mass * 0.4 * (lidar_radius * lidar_radius)}" ixy="0.0" ixz="0.0"
+        iyy="${lidar_mass * 0.4 * (lidar_radius * lidar_radius)}" iyz="0.0"
+        izz="${lidar_mass * 0.4 * (lidar_radius * lidar_radius)}"/>
+      </inertial>
+    </link>
+    <joint name="base_laser_joint" type="fixed">
+      <parent link="base_link"/>
+      <child link="base_laser"/>
+      <origin xyz="0.110 0 0.210" rpy="0 0 -1.5708"/>
+    </joint>
+    <joint name="camera_joint" type="fixed">
+        <parent link="base_link"/>
+        <child link="camera_link"/>
+        <origin xyz="0.225 0 0.140" rpy="0 0 0"/>
+    </joint>
+  <link name="camera_link">
+      <visual>
+          <geometry>
+              <box size="0.024 0.094 0.029"/>
+          </geometry>
+          <material name="black"/>
+      </visual>
+      <visual>
+          <origin xyz="0 0 -0.05"/>
+          <geometry>
+              <cylinder radius="0.002" length="0.1"/>
+          </geometry>
+          <material name="black"/>
+      </visual>
   </link>
-  <joint name="laser_joint" type="fixed">
-    <parent link="base_link"/>
-    <child link="laser_frame"/>
-    <!-- MODIFICAT: LiDAR pe Y (față) -->
-    <origin xyz="0 0.10 ${base_height + 0.0175}" rpy="0 0 0"/>
+  <joint name="camera_optical_joint" type="fixed">
+      <parent link="camera_link"/>
+      <child link="camera_link_optical"/>
+      <origin xyz="0 0 0" rpy="${-pi/2} 0 ${-pi/2}"/>
   </joint>
-  <!-- Include ros2_control -->
+  <link name="camera_link_optical"></link>
+  <!-- ============================================ -->
+  <!-- ROS2 CONTROL -->
+  <!-- ============================================ -->
   <xacro:dummybot_ros2_control
     name="DummyBotSystem"
@@ -134,5 +212,5 @@
     serial_baud="${serial_baud}"
     wheel_radius="${wheel_radius}"
-    wheel_separation="${wheel_separation}"
+    wheel_separation="${track_width}"
     ticks_per_revolution="${ticks_per_revolution}"/>
 </robot>

Commit message: Update URDF, controllers and sensor configurations
- Further URDF orientation fixes
- Updated diff_drive_controller parameters
- Added HD Pro Webcam C920 configuration
- Updated camera, LiDAR and sensors launch files
- Updated xplorer navigation config

File: ros2_ws/src/dummybot_bringup/description/urdf/dummybot.urdf.xacro (robot description, xacro)
@@ -162,5 +162,5 @@
         <cylinder length="${lidar_len}" radius="${lidar_radius}"/>
       </geometry>
-      <material name="white"/>
+      <material name="red"/>
     </visual>
     <inertial>
@@ -176,5 +176,5 @@
       <parent link="base_link"/>
       <child link="base_laser"/>
-      <origin xyz="0.110 0 0.210" rpy="0 0 -1.5708"/>
+      <origin xyz="0.110 0 0.210" rpy="0 0 0"/>
     </joint>
     <joint name="camera_joint" type="fixed">

Commit message: feat: nav2-semantic-route-server - YOLO26 dual-RPi + semantic localizer + route server + experiments

File: ros2_ws/src/dummybot_bringup/description/urdf/dummybot.urdf.xacro (robot description, xacro)
@@ -53,13 +53,13 @@
   <xacro:property name="ticks_per_revolution" value="1245"/>
   <!-- PID Controller Parameters (INT pentru ESP32, ordine: kp kd ki ko) -->
-  <xacro:property name="pid_kp" value="300"/>
-  <xacro:property name="pid_kd" value="70"/>
-  <xacro:property name="pid_ki" value="0"/>
-  <xacro:property name="pid_ko" value="14"/>
+  <xacro:property name="pid_kp" value="140"/>
+  <xacro:property name="pid_kd" value="20"/>
+  <xacro:property name="pid_ki" value="100"/>
+  <xacro:property name="pid_ko" value="20"/>
   <!-- Calibration Factors (FLOAT) -->
-  <xacro:property name="calibration_fl" value="0.875"/>
-  <xacro:property name="calibration_fr" value="1.065"/>
-  <xacro:property name="calibration_rl" value="1.025"/>
-  <xacro:property name="calibration_rr" value="1.025"/>
+  <xacro:property name="calibration_fl" value="1.0"/>
+  <xacro:property name="calibration_fr" value="1.0"/>
+  <xacro:property name="calibration_rl" value="1.0"/>
+  <xacro:property name="calibration_rr" value="1.0"/>
   <!-- Materials -->
   <material name="black">
